File: st-link.kicad_sch (KiCad schematic)
At the start: 38 parts, among them Q700 MMST3904, U700 STM32F103CBTx, Y700 8 MHz

Commit message: [rev 1.0] rev 1.0 finished
Other:
- title: ModuCard base module -> ModuCard nav module
Changed lines of the file:
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@@
 	(paper "A4")
 	(title_block
-		(title "ModuCard base module")
+		(title "ModuCard nav module")
 		(date "2025-02-18")
 		(rev "1.0.0")
 		(company "KoNaR")
 		(comment 1 "Base project authors: Dominik Pluta, Artem Horiunov")
-		(comment 2 "Project author: <author>")
+		(comment 2 "Project author: Patryk Dudziński")
 	)
 	(junction
